Commit message: Actualizacion 10-07

File: xacro/ackerman.xacro (robot description, xacro)
@@ -1,5 +1,5 @@
 <?xml version="1.0"?>
 <robot xmlns:xacro="http://www.ros.org/wiki/xacro">
-    <!--  -->
+    <!-- LINKS -->
     <!--Se incluyen los archivos xacro-->
     <xacro:include filename="base.xacro"/>
@@ -8,14 +8,15 @@
     <xacro:include filename="params.xacro"/>
     <!--Se agrega la base del robot-->
-    <xacro:base name="base_link" m="1500" w="${base_width}" l="${base_length}" h="${base_height}" zoff = "${zoff}"/>
+    <xacro:base name="base_link" m="${base_mass}" w="${base_width}" l="${base_length}" h="${base_height}" zoff = "${zoff}"/>
     <!--Voltantes del robot-->
-    <xacro:steering name="right_wheel_turn" m="1" rad="${steering_radius}" leng="${steering_length}"/>
-    <xacro:steering name="left_wheel_turn"  m="1" rad="${steering_radius}" leng="${steering_length}"/>
-    <xacro:steering name="steering_wheel"   m="1" rad="${steering_radius}" leng="${steering_length}"/>
+    <xacro:steering name="right_wheel_turn" m="${steering_mass}" rad="${steering_radius}" leng="${steering_length}"/>
+    <xacro:steering name="left_wheel_turn"  m="${steering_mass}" rad="${steering_radius}" leng="${steering_length}"/>
+    <xacro:steering name="steering_wheel"   m="${steering_mass}" rad="${steering_radius}" leng="${steering_length}"/>
     <!--Ruedas del robot-->
-    <xacro:wheel name="left_wheel_rear"     m="11" rad="${wheel_radius}" leng="${wheel_width}"/>
-    <xacro:wheel name="right_wheel_rear"    m="11" rad="${wheel_radius}" leng="${wheel_width}"/>
-    <xacro:wheel name="left_wheel_front"    m="11" rad="${wheel_radius}" leng="${wheel_width}"/>
-    <xacro:wheel name="right_wheel_front"   m="11" rad="${wheel_radius}" leng="${wheel_width}"/>
+    <xacro:wheel name="left_wheel_rear"     m="${wheel_mass}" rad="${wheel_radius}" leng="${wheel_width}"/>
+    <xacro:wheel name="right_wheel_rear"    m="${wheel_mass}" rad="${wheel_radius}" leng="${wheel_width}"/>
+    <xacro:wheel name="left_wheel_front"    m="${wheel_mass}" rad="${wheel_radius}" leng="${wheel_width}"/>
+    <xacro:wheel name="right_wheel_front"   m="${wheel_mass}" rad="${wheel_radius}" leng="${wheel_width}"/>
+    <!-- JOINTS -->
     <!--Enlace entre sistema de giro con rueda derecha superior-->
     <joint name="front_right_steer_joint" type="revolute">
@@ -24,5 +25,5 @@
         <child link="right_wheel_turn"/>
         <axis xyz="0.0 0.0 1.0"/>
-        <limit lower="-0.6458" upper="0.6458" effort="100" velocity="0.5"/>
+        <limit lower="${lower_limit}" upper="${upper_limit}" effort="100" velocity="0.5"/>
     </joint>
     <!--Enlace entre sistema de giro con rueda izquierda superior-->
@@ -32,5 +33,5 @@
         <child link="left_wheel_turn"/>
         <axis xyz="0.0 0.0 1.0"/>
-        <limit lower="-0.6458" upper="0.6458" effort="100" velocity="0.5"/>
+        <limit lower="${lower_limit}" upper="${upper_limit}" effort="100" velocity="0.5"/>
     </joint>
     <!--Enlace para el volante de dirección-->
@@ -69,13 +70,7 @@
         <axis xyz="0.0 1.0 0.0"/>
     </joint>
+    <!-- PLUGIN GAZENO ACKERMAN ROBOT -->
     <gazebo>
         <plugin name="gazebo_ros_ackermann_drive" filename="libgazebo_ros_ackermann_drive.so">
-            <!-- <ros>
-                <namespace>demo</namespace>
-                <remapping>cmd_vel:=cmd_demo</remapping>
-                <remapping>odom:=odom_demo</remapping>
-                <remapping>distance:=distance_demo</remapping>
-                <remapping>steerangle:=steerangle_demo</remapping>
-            </ros> -->
             <update_rate>400.0</update_rate>
             <!-- wheels -->

File: xacro/ackerman_plus.xacro (robot description, xacro)
@@ -1,4 +1,5 @@
 <?xml version="1.0"?>
 <robot xmlns:xacro="http://ros.org/wiki/xacro" name="ackerman_plus">
+    <!-- Funcion principal que hace llamado a los xacro -->
     <xacro:include filename="ackerman.xacro"/>
     <xacro:include filename="lidar.xacro"/>

File: xacro/params.xacro (robot description, xacro)
@@ -1,15 +1,22 @@
 <?xml version="1.0"?>
 <robot xmlns:xacro="http://ros.org/wiki/xacro">
+    <!-- Propiedades de la base -->
+    <xacro:property name="base_mass"    value = "1500"/>
     <xacro:property name="base_width"   value = "0.25"/>
     <xacro:property name="base_length"  value = "0.5"/>
     <xacro:property name="base_height"  value = "0.07"/>
+    <xacro:property name="zoff"         value = "0.15"/>
+    <!-- Propiedades de las ruedas -->
+    <xacro:property name="wheel_mass"   value = "11"/>
     <xacro:property name="wheel_radius" value = "0.1"/>
     <xacro:property name="wheel_width"  value = "0.05"/>
-    <xacro:property name="steering_radius" value = "0.05"/>
+    <!-- Propiedades de las direcciones -->
+    <xacro:property name="steering_mass"    value = "1"/>
+    <xacro:property name="steering_radius"  value = "0.05"/>
     <xacro:property name="steering_length"  value = "0.025"/>
-    <xacro:property name="zoff"  value = "0.15"/>
-    <xacro:property name="Green"  value = "0.0 1.0 0.0 1.0"/>
-    <xacro:property name="Black"  value = "0.0 0.0 0.0 1.0"/>
-    <!-- Define intertial property macros  -->
+    <!-- Limites superior e inferior ruedas -->
+    <xacro:property name="lower_limit" value = "-0.6458"/>
+    <xacro:property name="upper_limit" value = "0.6458"/>
+    <!-- Inercias de los objetos  -->
     <xacro:macro name="box_inertia" params="m w h l">
         <inertial>
