Commit message: Actualizacion 12-07

File: xacro/base.xacro (robot description, xacro)
@@ -1,5 +1,5 @@
 <?xml version="1.0"?>
 <robot xmlns:xacro="http://www.ros.org/wiki/xacro">
-    <!--Macro para las ruedas-->
+    <!--Macro para la base-->
     <xacro:macro name="base" params="name m w l h zoff">
     <link name="${name}">

File: xacro/camera.xacro (robot description, xacro)
@@ -1,48 +1,50 @@
 <?xml version="1.0"?>
 <robot xmlns:xacro="http://ros.org/wiki/xacro">
- <joint name="camera_joint" type="fixed">
-    <parent link="base_link"/>
-    <child link="camera_link"/>
-    <origin xyz="0.21 0 0.225" rpy="0 0 0"/>
- </joint>
- <link name="camera_link">
-    <visual>
-        <geometry>
-            <box size="0.01 0.03 0.03"/>
-        </geometry>
-        <material name="Blue">
-            <color rgba="0.0 0.0 1.0 1.0"/>
-        </material>
-    </visual>
-    <collision>
-        <geometry>
-            <box size="0.01 0.03 0.03"/>
-        </geometry>
-    </collision>
-    <inertial>
-        <origin xyz="0 0 0" rpy="${pi/2} 0 ${pi/2}"/>
-        <mass value="0.05"/>
-        <inertia ixx="${(0.05/12) * (0.03*0.03 + 0.03*0.03)}" ixy="0.0" ixz="0.0" iyy="${(0.05/12) * (0.01*0.01 + 0.03*0.03)}" iyz="0.0" izz="${(0.05/12) * (0.01*0.01 + 0.03*0.03)}"/>
-    </inertial>
- </link>
- <joint name="camera_optical_joint" type="fixed">
-    <parent link="camera_link"/>
-    <child link="camera_link_optical"/>
-    <origin xyz="0 0 0" rpy="${-pi/2} 0 ${-pi/2}"/>
- </joint>
- <link name="camera_link_optical">
- </link>
- <gazebo reference="camera_link">
-    <material>Gazebo/Red</material>
-    <sensor name="camera" type="camera" update_rate="10">
-        <pose>0 0 0 0 0 0</pose>
-        <visualize>true</visualize>
-        <camera>
-            <image width="320" height="240" hfov="1.5708" format="RGB8" near="0.0"/>
-        </camera>
-        <plugin name="camera_controller" filename="libgazebo_ros_camera.so">
-            <frame_name>camera_link_optical</frame_name>
-        </plugin>
-    </sensor>
- </gazebo>
+    <!-- Macro para la camara -->
+    <!-- Enlace entre la camara y el robot -->
+    <joint name="camera_joint" type="fixed">
+        <parent link="base_link"/>
+        <child link="camera_link"/>
+        <origin xyz="0.21 0 0.225" rpy="0 0 0"/>
+    </joint>
+    <link name="camera_link">
+        <visual>
+            <geometry>
+                <box size="0.01 0.03 0.03"/>
+            </geometry>
+            <material name="Blue">
+                <color rgba="0.0 0.0 1.0 1.0"/>
+            </material>
+        </visual>
+        <collision>
+            <geometry>
+                <box size="0.01 0.03 0.03"/>
+            </geometry>
+        </collision>
+        <inertial>
+            <origin xyz="0 0 0" rpy="${pi/2} 0 ${pi/2}"/>
+            <mass value="0.05"/>
+            <inertia ixx="${(0.05/12) * (0.03*0.03 + 0.03*0.03)}" ixy="0.0" ixz="0.0" iyy="${(0.05/12) * (0.01*0.01 + 0.03*0.03)}" iyz="0.0" izz="${(0.05/12) * (0.01*0.01 + 0.03*0.03)}"/>
+        </inertial>
+    </link>
+    <joint name="camera_optical_joint" type="fixed">
+        <parent link="camera_link"/>
+        <child link="camera_link_optical"/>
+        <origin xyz="0 0 0" rpy="${-pi/2} 0 ${-pi/2}"/>
+    </joint>
+    <link name="camera_link_optical">
+    </link>
+    <gazebo reference="camera_link">
+        <material>Gazebo/Red</material>
+        <sensor name="camera" type="camera" update_rate="10">
+            <pose>0 0 0 0 0 0</pose>
+            <visualize>true</visualize>
+            <camera>
+                <image width="320" height="240" hfov="1.5708" format="RGB8" near="0.0"/>
+            </camera>
+            <plugin name="camera_controller" filename="libgazebo_ros_camera.so">
+                <frame_name>camera_link_optical</frame_name>
+            </plugin>
+        </sensor>
+    </gazebo>
 </robot>

File: xacro/lidar.xacro (robot description, xacro)
@@ -1,4 +1,6 @@
 <?xml version="1.0"?>
 <robot xmlns:xacro="http://www.ros.org/wiki/xacro">
+    <!-- Macro para el sensor de tipo lidar -->
+    <!-- Enlace entre el sensor y el robot -->
     <joint name="laser_joint" type="fixed">
         <parent link="base_link"/>
@@ -25,8 +27,8 @@
         <material>Gazebo/Red</material>
         <sensor name="laser" type="ray">
-            <pose> 0 0 0 0 0 0 </pose> <!-- Origen de sensor -->
-            <visualize> false </visualize> <!-- Visualizacion de sensor -->
-            <update_rate> 10 </update_rate> <!-- 1 Hz -->
-            <ray> <!-- Parametros de sensor virtual -->
+            <pose> 0 0 0 0 0 0 </pose>
+            <visualize> false </visualize>
+            <update_rate> 10 </update_rate>
+            <ray>
                 <scan>
                     <horizontal>

File: xacro/steering.xacro (robot description, xacro)
@@ -1,5 +1,5 @@
 <?xml version="1.0"?>
 <robot xmlns:xacro="http://www.ros.org/wiki/xacro">
-    <!--Macro para las ruedas-->
+    <!--Macro para los volante-->
     <xacro:macro name="steering" params="name m rad leng">
     <link name="${name}">
